Commit message: 更正了一些配置，完善笔记

File: ros_ws/src/vehicle_description/urdf/out.urdf (robot description, URDF)
Before this commit: robot hrbot, 9 links, 8 joints
Joints:
- joint wheel_1_joint: type continuous -> fixed
- joint wheel_2_joint: type continuous -> fixed
- joint wheel_3_joint: type continuous -> fixed
- joint wheel_4_joint: type continuous -> fixed

Commit message: 修改车辆urdf描述文件、删除nav下多余的move.py和地图文件、删除stm32下多余的i2c程序、mission下新增teb算法和交通灯识别

File: ros_ws/src/vehicle_description/urdf/out.urdf (robot description, URDF)
Before this commit: robot hrbot, 9 links, 8 joints
Joints:
- joint wheel_1_joint: origin xyz=0.1 0.14 -0.02 rpy=0 0 0 -> xyz=0.16 0.14 -0.02 rpy=0 0 0
- joint wheel_2_joint: origin xyz=0.1 -0.14 -0.02 rpy=0 0 0 -> xyz=0.16 -0.14 -0.02 rpy=0 0 0
- joint wheel_3_joint: origin xyz=-0.1 0.14 -0.02 rpy=0 0 0 -> xyz=-0.16 0.14 -0.02 rpy=0 0 0
- joint wheel_4_joint: origin xyz=-0.1 -0.14 -0.02 rpy=0 0 0 -> xyz=-0.16 -0.14 -0.02 rpy=0 0 0
